File: NodeMCU_watering_system.sch (EAGLE design)
At the start: 24 parts, among them IC1 7805DT

Commit message: Add files via upload
Parts:
- removed REL1, REL2: RR1A, #PaJa_22:RR1A
- added JP9: (no value), SparkFun:M03LONGPADS
- added R7, R8: 4k7, rcl:R-EU_M0805
- added REL3, REL4: RELSIA, #PaJa_22:RELSIA
- C1, C2: value (none) -> 100n
- JP4: value valve -> ouput1
- JP5: value pump -> output2
- JP6: value On/Off -> output1LED
- JP7: value valve on -> ouput2LED
- JP8: value Vin IN -> VIN
- Q1, Q2: value (none) -> IRLML2520
- R1, R3: value 10k -> 1K
- R2, R4: value 10k -> 33K
- R5, R6: value (none) -> 820R
Connections:
- removed net PUMP: R3.1
- removed net VALVE: R1.1
- new net N$10: D1.K, D2.K, JP9.2, REL3CIVKA.C+, REL4CIVKA.C+
- new net OUTPUT1: R1.1, U$1.D5
- new net OUTPUT2: R3.1, U$1.D6
- net 3V3: now also R7.2, R8.2, U$1.3V3@2
- net 5V: now also JP9.1, U$1.VIN; no longer D1.K, D2.K, REL1CIVKA.C+, REL2CIVKA.C+
- net GND: now also U$1.GND@1; no longer U$1.GND@0
- net N$4: now also REL3CIVKA.C-; no longer REL1CIVKA.C-
- net N$5: now also REL4CIVKA.C-; no longer REL2CIVKA.C-
- net N$6: now also REL3SPIN.2; no longer REL1SPINAC.2
- net N$7: now also REL4SPIN.2; no longer REL2SPINAC.2
- net SCL: now also R7.1
- net SDA: now also R8.1
- net VIN: now also JP9.3, REL3SPIN.1, REL4SPIN.1; no longer REL1SPINAC.1, REL2SPINAC.1, U$1.VIN

Commit message: Add files via upload
Parts:
- JP4: value ouput1 -> output1
Changed lines of the file:
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@@
 <?xml version="1.0" encoding="utf-8"?>
 <!DOCTYPE eagle SYSTEM "eagle.dtd">
-<eagle version="7.6.0">
+<eagle version="8.2.0">
 <drawing>
 <settings>
@@
 <part name="R5" library="rcl" deviceset="R-EU_" device="M0805" value="820R"/>
 <part name="R6" library="rcl" deviceset="R-EU_" device="M0805" value="820R"/>
-<part name="JP4" library="SparkFun" deviceset="M02" device="LOCK_LONGPADS" value="ouput1"/>
+<part name="JP4" library="SparkFun" deviceset="M02" device="LOCK_LONGPADS" value="output1"/>
 <part name="JP5" library="SparkFun" deviceset="M02" device="LOCK_LONGPADS" value="output2"/>
 <part name="D1" library="#PaJa_30" deviceset="1N4007" device="_SM-1"/>
